File: schematics/circuit/wordclock-0.1/wordclock.kicad_sch (KiCad schematic)
At the start: 14 parts, among them U1 STM32F303RCTx, Y1 32.768kHz, Y2 8MHz

Commit message: Initial 16x16 wordclock layout
Parts:
- R1: footprint (none) -> Resistor_SMD:R_1210_3225Metric
Changed lines of the file:
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@@
       (effects (font (size 1.27 1.27)))
     )
-    (property "Footprint" "" (at 46.99 167.132 90)
+    (property "Footprint" "Resistor_SMD:R_1210_3225Metric" (at 46.99 167.132 90)
       (effects (font (size 1.27 1.27)) hide)
     )
