File: schematics/circuit/wordclock-0.1/wordclock.kicad_pcb (KiCad board)
At the start: 2 copper layers, 282 parts, among them U1 STM32F303RCTx, U2 MAX7219, U3 MAX7219, U4 MAX7219, U5 MAX7219, Y1 32.768kHz, Y2 8MHz

Commit message: Change tracked files
Parts:
- C1, C10, C11, C12, C13, C14, C2, C3, C4, C5, C6, C7, C8, C9, R1, R2, R3, R4, R5, U1, U2, U3, U4, U5, Y1, Y2: moved to B.Cu
- moved U5 287.3 mm to (464.8, 328.3), turned to 180 degrees
- moved R5 263.0 mm to (474.1, 337.8), turned to 180 degrees
- moved C14 257.1 mm to (478.5, 337.9), turned to 180 degrees
- moved C13 230.2 mm to (365.8, 342.9), turned to 180 degrees
- moved U4 227.0 mm to (370.3, 328.3), turned to 180 degrees
- moved R4 221.8 mm to (357.2, 342.9)
- moved C12 203.6 mm to (504.5, 335.3), turned to 180 degrees
- moved R3 192.4 mm to (499.5, 335.3), turned to 180 degrees
- moved U2 190.6 mm to (417.6, 328.3), turned to 180 degrees
- moved R2 179.6 mm to (392.8, 340.4), turned to 180 degrees
- moved U1 173.8 mm to (442.0, 358.1), turned to -135 degrees
- moved C11 173.5 mm to (402.9, 340.4), turned to 180 degrees
- moved U3 142.7 mm to (512.1, 328.3), turned to 180 degrees
- moved R1 117.6 mm to (468.8, 381.0), turned to 180 degrees
- moved Y1 115.3 mm to (440.5, 376.8), turned to 180 degrees
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