File: schematics/circuit/wordclock-0.0.1/wordclock.kicad_pcb (KiCad board)
At the start: 2 copper layers, 282 parts, among them U1 STM32F303RCTx, U2 MAX7219, U3 MAX7219, U4 MAX7219, U5 MAX7219, Y1 32.768kHz, Y2 8MHz

Commit message: Initial pcb layout
Parts:
- added BT1: Battery_Cell, Battery:BatteryHolder_Keystone_3002_1x2032, B.Cu at (499.3, 221.4)
- added C11: 100nF, Capacitor_SMD:C_0402_1005Metric, B.Cu at (442.2, 236.3)
- added C12: 100nF, Capacitor_SMD:C_0402_1005Metric, B.Cu at (443.5, 236.3)
- added C13: 10uF, Capacitor_SMD:C_0805_2012Metric, B.Cu at (417.4, 407.7)
- added C14: 1uF, Capacitor_SMD:C_0402_1005Metric, B.Cu at (456.2, 218.9)
- added C15: 0.1uF, Capacitor_SMD:C_0402_1005Metric, B.Cu at (456.2, 220.9)
- added C16: 10nF, Capacitor_SMD:C_0603_1608Metric, B.Cu at (422.7, 401.1)
- added C17: ?, Capacitor_SMD:C_0603_1608Metric, B.Cu at (429.1, 397.5)
- added C18: 68uF, Capacitor_SMD:C_0603_1608Metric, B.Cu at (431.6, 400.5)
- added D500: Status, LED_SMD:LED_0603_1608Metric, B.Cu at (441.1, 209.8)
- added D501: SHCK, Diode_SMD:D_SOD-123, B.Cu at (421.0, 411.8)
- added F1: 1A, Fuse:Fuse_1206_3216Metric, B.Cu at (418.1, 415.6)
- added FB1: 600 @ 600MHz, Inductor_SMD:L_0805_2012Metric, B.Cu at (421.0, 407.0)
- added H1: MountingHole_Pad, MountingHole:MountingHole_4.3mm_M4_Pad_Via, F.Cu at (274.3, 54.0)
- added H2: MountingHole_Pad, MountingHole:MountingHole_4.3mm_M4_Pad_Via, F.Cu at (274.1, 385.8)
- added H3: MountingHole_Pad, MountingHole:MountingHole_4.3mm_M4_Pad_Via, F.Cu at (609.6, 51.5)
- added H4: MountingHole_Pad, MountingHole:MountingHole_4.3mm_M4_Pad_Via, F.Cu at (607.1, 386.8)
- added J1: TagConnect, Connector:Tag-Connect_TC2030-IDC-FP_2x03_P1.27mm_Vertical, B.Cu at (439.2, 197.6)
- added L1: 39nH, Inductor_SMD:L_Sunlord_MWSA0518S, B.Cu at (474.5, 424.3)
- added L2: 3.3uH, Inductor_SMD:L_0402_1005Metric, B.Cu at (428.6, 403.1)
- added P1: USB_C_Plug, Connector_USB:USB_C_Receptacle_GCT_USB4115-03-C, B.Cu at (428.1, 413.5)
- added Q1: AO3401A, Package_TO_SOT_SMD:SOT-23, B.Cu at (417.5, 412.2)
- added R10: 10k, Resistor_SMD:R_0805_2012Metric, B.Cu at (425.5, 397.5)
- added R11: 22, Resistor_SMD:R_0603_1608Metric, B.Cu at (446.4, 196.5)
- added R12: 22, Resistor_SMD:R_0603_1608Metric, B.Cu at (446.4, 199.0)
- added R2: 47Ω, Resistor_SMD:R_0402_1005Metric, B.Cu at (403.9, 218.4)
- added R3: 242k, Resistor_SMD:R_0805_2012Metric, B.Cu at (424.4, 218.6)
- added R4: 1k5, Resistor_SMD:R_0402_1005Metric, B.Cu at (438.3, 209.7)
- added R5: 100k, Resistor_SMD:R_0805_2012Metric, B.Cu at (418.5, 404.5)
- added R6: 68k, Resistor_SMD:R_0805_2012Metric, B.Cu at (416.1, 404.5)
- added R7: 4.7k, Resistor_SMD:R_0402_1005Metric, B.Cu at (449.4, 425.3)
- added R8: 4.7k, Resistor_SMD:R_0402_1005Metric, B.Cu at (449.4, 427.3)
- added R9: 31.25k, Resistor_SMD:R_0805_2012Metric, B.Cu at (428.5, 400.7)
- added SW1: SW_SPDT, Button_Switch_SMD:SW_SPDT_PCM12, B.Cu at (479.1, 408.9)
- added U6: USBLC6-2SC6, Package_TO_SOT_SMD:SOT-23-6, B.Cu at (431.0, 408.2)
- added U7: ~, Package_TO_SOT_SMD:SOT-23-6, B.Cu at (425.5, 401.1)
- added U8: DS3231MZ, Package_SO:SOIC-8_3.9x4.9mm_P1.27mm, B.Cu at (461.8, 219.4)
- added U9: AT24CS02-SSHM, Package_SO:SOIC-8_3.9x4.9mm_P1.27mm, B.Cu at (391.0, 220.4)
- C1: value 10pF -> 4.7uF; footprint Capacitor_SMD:C_0805_2012Metric -> Capacitor_SMD:C_0603_1608Metric
- C10, C6: footprint Capacitor_SMD:C_0805_2012Metric -> Capacitor_SMD:C_0402_1005Metric
- C2: footprint Capacitor_SMD:C_0805_2012Metric -> Capacitor_SMD:C_0603_1608Metric
- C3: value 20pF -> 12pF; footprint Capacitor_SMD:C_0805_2012Metric -> Capacitor_SMD:C_0603_1608Metric
- C4: value 10pF -> 1uF; footprint Capacitor_SMD:C_0805_2012Metric -> Capacitor_SMD:C_0402_1005Metric
- C5: value 1uF -> 100nF; footprint Capacitor_SMD:C_0805_2012Metric -> Capacitor_SMD:C_0402_1005Metric
- C7: value 4.7uF -> 100nF; footprint Capacitor_SMD:C_0805_2012Metric -> Capacitor_SMD:C_0402_1005Metric
- C8: value 100nF -> 12pF; footprint Capacitor_SMD:C_0805_2012Metric -> Capacitor_SMD:C_0603_1608Metric
- C9: value 100nF -> 20pF; footprint Capacitor_SMD:C_0805_2012Metric -> Capacitor_SMD:C_0603_1608Metric
- R1: value 0 -> 10k; footprint Resistor_SMD:R_1210_3225Metric -> Resistor_SMD:R_0603_1608Metric
- Y1: value 32.768kHz -> 8MHz
- Y2: value 8MHz -> 32.768kHz
- moved C21 181.1 mm to (470.9, 195.5), turned to -90 degrees
- moved R15 180.4 mm to (470.0, 202.1), turned to 90 degrees
- moved C8 171.1 mm to (404.7, 220.8)
- moved C2 170.8 mm to (424.4, 214.2)
- moved C3 170.7 mm to (402.3, 223.7)
- moved Y2 169.1 mm to (420.0, 219.1)
- moved C9 166.5 mm to (424.5, 223.6)
- moved Y1 162.3 mm to (400.5, 219.4)
- moved D100 160.0 mm to (370.0, 290.0)
- moved D101 160.0 mm to (370.0, 310.0)
- moved D102 160.0 mm to (370.0, 330.0)
- moved D103 160.0 mm to (370.0, 350.0)
- moved D104 160.0 mm to (370.0, 370.0)
- moved D105 160.0 mm to (390.0, 230.0)
- moved D106 160.0 mm to (390.0, 250.0)
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- renumbered C11 to C19, C12 to C20, C13 to C21, C14 to C22, R2 to R13, R3 to R14, R4 to R15, R5 to R16, U2 to U1, U3 to U2, U4 to U3, U5 to U4, U1 to U5
Connections:
- net /CLK renamed SPI2_CLK
- net /LOAD renamed SPI2_LOAD
- net /MISO renamed SPI2_MISO
- net /MOSI renamed SPI2_MOSI
- C1 pad 1: Earth -> CLOCK_VCC
- C1 pad 2: Net-(U1-PC14) -> GND
- C10 pad 1: VDD -> CLOCK_VCC
- C10 pad 2: Earth -> GND
- C19 pad 1: VDD -> CLOCK_VCC
- C2 pad 1: Earth -> OSC32_IN
- C2 pad 2: Net-(U1-PF0) -> GND
- C20 pad 1: VDD -> CLOCK_VCC
- C21 pad 1: VDD -> CLOCK_VCC
- C22 pad 1: VDD -> CLOCK_VCC
- C3 pad 1: Earth -> OSC_IN
- C3 pad 2: Net-(U1-PF1) -> GND
- C4 pad 1: Net-(C4-Pad1) -> +3.3VA
- C4 pad 2: Earth -> GND
- C5 pad 1: VDDA -> CLOCK_VCC
- C5 pad 2: Earth -> GND
- C6 pad 1: VDDA -> +3.3VA
- C6 pad 2: Earth -> GND
- C7 pad 1: VDD -> CLOCK_VCC
- C7 pad 2: Earth -> GND
- C8 pad 1: VDD -> Net-(C8-Pad1)
- C8 pad 2: Earth -> GND
- C9 pad 1: VDD -> Net-(C9-Pad1)
- C9 pad 2: Earth -> GND
- R1 pad 1: Net-(U1-PC15) -> BOOT0
- R1 pad 2: Net-(C4-Pad1) -> Net-(SW1-B)
- R13 pad 2: VDD -> CLOCK_VCC
- R14 pad 2: VDD -> CLOCK_VCC
- R15 pad 2: VDD -> CLOCK_VCC
- R16 pad 2: VDD -> CLOCK_VCC
- U1 pad 19: VDD -> CLOCK_VCC
- U2 pad 19: VDD -> CLOCK_VCC
- U3 pad 19: VDD -> CLOCK_VCC
- U4 pad 19: VDD -> CLOCK_VCC
- U5 pad 1: unconnected-(U1-VBAT-Pad1) -> CLOCK_VCC
- U5 pad 12: unconnected-(U1-VSSA-Pad12) -> GND
- U5 pad 13: unconnected-(U1-VDDA-Pad13) -> +3.3VA
- U5 pad 16: unconnected-(U1-PA2-Pad16) -> LED_STATUS
- U5 pad 19: unconnected-(U1-VDD-Pad19) -> CLOCK_VCC
- U5 pad 3: Net-(U1-PC14) -> OSC32_IN
- U5 pad 31: Earth -> GND
- U5 pad 32: unconnected-(U1-VDD-Pad32) -> CLOCK_VCC
- U5 pad 4: Net-(U1-PC15) -> OSC32_OUT
- U5 pad 44: unconnected-(U1-PA11-Pad44) -> USB_D-
- U5 pad 45: unconnected-(U1-PA12-Pad45) -> USB_D+
- U5 pad 46: unconnected-(U1-PA13-Pad46) -> SWDIO
- U5 pad 47: Earth -> GND
- U5 pad 48: unconnected-(U1-VDD-Pad48) -> CLOCK_VCC
- U5 pad 49: unconnected-(U1-PA14-Pad49) -> SWCLK
- U5 pad 5: Net-(U1-PF0) -> OSC_IN
- U5 pad 55: unconnected-(U1-PB3-Pad55) -> TRACESWO
- U5 pad 59: unconnected-(U1-PB7-Pad59) -> I2C1_SDA
- U5 pad 6: Net-(U1-PF1) -> OSC_OUT
- U5 pad 60: unconnected-(U1-BOOT0-Pad60) -> BOOT0
- U5 pad 61: unconnected-(U1-PB8-Pad61) -> I2C1_SCL
- U5 pad 63: Earth -> GND
- U5 pad 64: unconnected-(U1-VDD-Pad64) -> CLOCK_VCC
- U5 pad 7: unconnected-(U1-NRST-Pad7) -> NRST
- Y1 pad 1: Net-(C4-Pad1) -> OSC_IN
- Y1 pad 2: Net-(U1-PC14) -> GND
- Y1 pad 3: (no net) -> Net-(C8-Pad1)
- Y1 pad 4: (no net) -> GND
- Y2 pad 1: Net-(U1-PF1) -> OSC32_IN
- Y2 pad 2: Net-(U1-PF0) -> GND
- Y2 pad 3: (no net) -> Net-(C9-Pad1)
- Y2 pad 4: (no net) -> GND
Routing:
- net /Led Array 3/row0: track 0.00 -> 281.4 mm, vias 0 -> 1
- net /Led Array 4/row0: track 0.00 -> 280.7 mm, vias 0 -> 1
- net /Led Array 3/col7: track 0.00 -> 279.6 mm, vias 0 -> 1
- net /Led Array 4/col0: track 0.00 -> 277.6 mm, vias 0 -> 1
- net /Led Array 3/row1: track 0.00 -> 262.2 mm, vias 0 -> 10
- net /Led Array 4/row1: track 0.00 -> 261.8 mm, vias 0 -> 9
- net /Led Array 3/col6: track 0.00 -> 254.0 mm, vias 0 -> 1
- net /Led Array 4/col1: track 0.00 -> 245.7 mm, vias 0 -> 1
- net /Led Array 3/row2: track 0.00 -> 242.5 mm, vias 0 -> 10
- net /Led Array 3/col5: track 0.00 -> 242.4 mm, vias 0 -> 1
- net /Led Array 4/row2: track 0.00 -> 241.9 mm, vias 0 -> 9
- net /Led Array 4/col2: track 0.00 -> 233.0 mm, vias 0 -> 1
- net /Led Array 4/row3: track 0.00 -> 224.3 mm, vias 0 -> 9
- net /Led Array 3/row3: track 0.00 -> 223.9 mm, vias 0 -> 10
- net /Led Array 3/col4: track 0.00 -> 211.6 mm, vias 0 -> 1
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Other:
- copper layers 2 -> 4
