File: schematics/circuit/wordclock-proto-r1/wordclock-proto-r1.kicad_pcb (KiCad board)
At the start: 4 copper layers, 198.8 x 160 mm, 115 parts, among them J1 TagConnect, P1 USB_C_Plug, Q1 AO3401A, SW1 SW_SPDT, U1 MAX7219, U5 STM32F303RCTx, U6 USBLC6-2SC6, U8 DS3231MZ, U9 AT24CS02-SSHM, Y1 8MHz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

Commit message: more pcb changes
Parts:
- removed U6: USBLC6-2SC6, Package_TO_SOT_SMD:SOT-23-6
- moved R8 100.9 mm to (163.2, 90.6), turned to -90 degrees
- moved R7 96.3 mm to (166.0, 95.1), turned to 0 degrees
- moved C6 81.3 mm to (169.1, 115.3), turned to -90 degrees
- moved C4 79.7 mm to (170.4, 115.3), turned to -90 degrees
- moved BT1 79.2 mm to (141.4, 88.8), turned to 0 degrees
- moved C15 77.6 mm to (172.2, 90.6), turned to 90 degrees
- moved U7 77.6 mm to (185.1, 118.0), turned to 0 degrees
- moved C14 75.7 mm to (173.5, 90.6), turned to 90 degrees
- moved R10 75.5 mm to (179.5, 116.7), turned to 90 degrees
- moved R9 73.1 mm to (181.7, 116.6), turned to 90 degrees
- moved L2 72.4 mm to (186.3, 121.1), turned to -90 degrees
- moved F1 71.1 mm to (186.2, 110.7), turned to -90 degrees
- moved D501 66.5 mm to (190.1, 108.0), turned to 0 degrees
- moved C17 65.3 mm to (183.8, 114.4), turned to -90 degrees
- moved R5 65.2 mm to (189.6, 117.0), turned to 0 degrees
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Connections:
- P1 pad A6: USB_CONN_D+ -> unconnected-(P1-D+-PadA6)
- P1 pad A7: USB_CONN_D- -> unconnected-(P1-D--PadA7)
- U5 pad 44: USB_D- -> unconnected-(U5-PA11-Pad44)
- U5 pad 45: USB_D+ -> unconnected-(U5-PA12-Pad45)
Routing:
- net GND: track 25.6 -> 136.3 mm, vias 4 -> 36
- net /Led Array 1/col7: track 140.0 -> 201.4 mm, vias 0 -> 3
- net +BATT: track 0.00 -> 53.2 mm
- net /Led Array 1/col3: track 215.9 -> 172.2 mm
- net /Led Array 1/col2: track 233.9 -> 191.2 mm
- net /Led Array 1/col4: track 188.9 -> 146.5 mm
- net /Led Array 1/col0: track 266.9 -> 225.7 mm
- net +3.3V: track 9.46 -> 50.3 mm, vias 1 -> 18
- net /Led Array 1/col1: track 259.5 -> 218.9 mm
- net BOOT0: track 0.00 -> 35.5 mm
- net /Led Array 1/col6: track 150.5 -> 182.3 mm, vias 1 -> 3
- net /Led Array 1/col5: track 177.8 -> 149.2 mm
- net TRACESWO: track 0.00 -> 26.8 mm, vias 0 -> 2
- net SWCLK: track 0.00 -> 24.7 mm, vias 0 -> 2
- net NRST: track 0.00 -> 24.4 mm, vias 0 -> 2
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- added copper zone on In1.Cu, net +3.3V
- added copper zone on In2.Cu, net GND
Other:
- board size 198.8 x 160 mm -> 160 x 160 mm
- board text added: "JLCJLCJLCJLC"
