File: schematics/circuit/wordclock-proto-r1/wordclock-proto-r1.kicad_sch (KiCad schematic)
At the start: 52 parts, among them J1 TagConnect, P1 USB_C_Plug, Q1 AO3401A, SW1 SW_SPDT, U5 STM32F303RCTx, U6 USBLC6-2SC6, U8 DS3231MZ, U9 AT24CS02-SSHM, Y1 8MHz, Y2 32.768kHz

Commit message: Add prototype board project
Parts:
- removed H1, H2, H3, H4: MountingHole_Pad, MountingHole:MountingHole_4.3mm_M4_Pad_Via, symbol Mechanical:MountingHole_Pad
- C2, C3, C8, C9: footprint Capacitor_SMD:C_0603_1608Metric -> Capacitor_SMD:C_0402_1005Metric
- R3: footprint Resistor_SMD:R_0805_2012Metric -> Resistor_SMD:R_0402_1005Metric
Connections:
- net +5V: now also Q1.3 (D); no longer F1.1
- net at F1.2: now also FB1.1; no longer Q1.3 (D)
- net at D501.1 (K), Q1.2 (S): now also F1.1; no longer FB1.1
Other:
- removed sheet Led Array 2
- removed sheet Led Array 3
- removed sheet Led Array 4
- moved on the sheet: D501, F1, Q1

Commit message: more pcb changes
Parts:
- removed U6: USBLC6-2SC6, Package_TO_SOT_SMD:SOT-23-6, symbol Power_Protection:USBLC6-2SC6
Connections:
- net USB_CONN_D+: no longer names the net of P1.A6 (D+)
- net USB_CONN_D-: no longer names the net of P1.A7 (D-)
- net USB_D+: no longer names the net of U5.45 (PA12)
- net USB_D-: no longer names the net of U5.44 (PA11)
- no-connect marks 55 -> 59
Changed lines of the file:
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@@
   (no_connect (at 48.26 52.705))
   (no_connect (at 192.405 190.5))
+  (no_connect (at 227.965 149.86))
   (no_connect (at 295.91 266.065))
   (no_connect (at 227.965 121.92))
@@
   (no_connect (at 192.405 195.58))
   (no_connect (at 48.26 32.385))
+  (no_connect (at 48.26 42.545))
   (no_connect (at 192.405 187.96))
   (no_connect (at 227.965 139.7))
@@
   (no_connect (at 355.6 212.09))
   (no_connect (at 192.405 193.04))
+  (no_connect (at 48.26 37.465))
   (no_connect (at 192.405 180.34))
   (no_connect (at 192.405 198.12))
@@
   (no_connect (at 48.26 57.785))
   (no_connect (at 48.26 83.185))
+  (no_connect (at 227.965 152.4))
   (no_connect (at 227.965 142.24))
   (no_connect (at 48.26 29.845))
@@
     (stroke (width 0) (type default))
   )
-  (wire (pts (xy 118.745 81.915) (xy 118.745 84.455))
-    (stroke (width 0) (type default))
-  )
   (wire (pts (xy 365.76 222.25) (xy 365.76 223.52))
     (stroke (width 0) (type default))
@@
     (stroke (width 0) (type default))
   )
-  (wire (pts (xy 118.745 59.69) (xy 118.745 61.595))
-    (stroke (width 0) (type default))
-  )
   (wire (pts (xy 25.4 255.905) (xy 25.4 242.57))
     (stroke (width 0) (type default))
@@
     )
   )
-  (global_label "USB_D+" (shape input) (at 227.965 152.4 0) (fields_autoplaced)
-    (effects (font (size 1.27 1.27)) (justify left))
-    (property "Intersheetrefs" "${INTERSHEET_REFS}" (at 238.4908 152.4 0)
-      (effects (font (size 1.27 1.27)) (justify left) hide)
-    )
-  )
-  (global_label "USB_D-" (shape input) (at 108.585 69.215 180) (fields_autoplaced)
-    (effects (font (size 1.27 1.27)) (justify right))
-    (property "Intersheetrefs" "${INTERSHEET_REFS}" (at 98.0592 69.215 0)
-      (effects (font (size 1.27 1.27)) (justify right) hide)
-    )
-  )
   (global_label "I2C1_SDA" (shape input) (at 270.51 260.985 180) (fields_autoplaced)
     (effects (font (size 1.27 1.27)) (justify right))
@@
     )
   )
-  (global_label "USB_D-" (shape input) (at 227.965 149.86 0) (fields_autoplaced)
-    (effects (font (size 1.27 1.27)) (justify left))
-    (property "Intersheetrefs" "${INTERSHEET_REFS}" (at 238.4908 149.86 0)
-      (effects (font (size 1.27 1.27)) (justify left) hide)
-    )
-  )
   (global_label "SPI2_MOSI" (shape input) (at 377.825 26.035 180) (fields_autoplaced)
     (effects (font (size 1.27 1.27)) (justify right))
@@
     )
   )
-  (global_label "USB_D+" (shape input) (at 128.905 69.215 0) (fields_autoplaced)
-    (effects (font (size 1.27 1.27)) (justify left))
-    (property "Intersheetrefs" "${INTERSHEET_REFS}" (at 139.4308 69.215 0)
-      (effects (font (size 1.27 1.27)) (justify left) hide)
-    )
-  )
   (global_label "BUCK_EN" (shape input) (at 246.38 36.83 180) (fields_autoplaced)
     (effects (font (size 1.27 1.27)) (justify right))
@@
     )
   )
-  (global_label "USB_CONN_D+" (shape input) (at 128.905 74.295 0) (fields_autoplaced)
-    (effects (font (size 1.27 1.27)) (justify left))
-    (property "Intersheetrefs" "${INTERSHEET_REFS}" (at 145.6599 74.295 0)
-      (effects (font (size 1.27 1.27)) (justify left) hide)
-    )
-  )
   (global_label "SPI2_LOAD" (shape input) (at 227.965 195.58 0) (fields_autoplaced)
     (effects (font (size 1.27 1.27)) (justify left))
@@
     )
   )
-  (global_label "USB_CONN_D-" (shape input) (at 48.26 37.465 0) (fields_autoplaced)
-    (effects (font (size 1.27 1.27)) (justify left))
-    (property "Intersheetrefs" "${INTERSHEET_REFS}" (at 65.0149 37.465 0)
-      (effects (font (size 1.27 1.27)) (justify left) hide)
-    )
-  )
   (global_label "BUCK_FB" (shape input) (at 264.16 36.83 0) (fields_autoplaced)
     (effects (font (size 1.27 1.27)) (justify left))
@@
     )
   )
-  (global_label "USB_CONN_D+" (shape input) (at 48.26 42.545 0) (fields_autoplaced)
-    (effects (font (size 1.27 1.27)) (justify left))
-    (property "Intersheetrefs" "${INTERSHEET_REFS}" (at 65.0149 42.545 0)
-      (effects (font (size 1.27 1.27)) (justify left) hide)
-    )
-  )
   (global_label "SWDIO" (shape input) (at 352.425 135.255 90) (fields_autoplaced)
     (effects (font (size 1.27 1.27)) (justify left))
@@
     )
   )
-  (global_label "USB_CONN_D-" (shape input) (at 108.585 74.295 180) (fields_autoplaced)
-    (effects (font (size 1.27 1.27)) (justify right))
-    (property "Intersheetrefs" "${INTERSHEET_REFS}" (at 91.8301 74.295 0)
-      (effects (font (size 1.27 1.27)) (justify right) hide)
-    )
-  )
   (global_label "SWCLK" (shape input) (at 227.965 157.48 0) (fields_autoplaced)
     (effects (font (size 1.27 1.27)) (justify left))
@@
     )
   )
-  (symbol (lib_id "power:GND") (at 118.745 84.455 0) (unit 1)
-    (in_bom yes) (on_board yes) (dnp no)
-    (property "Reference" "#PWR0132" (at 118.745 90.805 0)
-      (effects (font (size 1.27 1.27)) hide)
-    )
-    (property "Value" "GND" (at 118.745 88.265 0)
-      (effects (font (size 1.27 1.27)))
-    )
-    (property "Footprint" "" (at 118.745 84.455 0)
-      (effects (font (size 1.27 1.27)) hide)
-    )
-    (property "Datasheet" "" (at 118.745 84.455 0)
-      (effects (font (size 1.27 1.27)) hide)
-    )
-    (pin "1")
-    (instances
-      (project "wordclock-proto-r1"
-        (path "/4f94f353-fcb1-446a-8ea4-44fbed72b7d1"
-          (reference "#PWR0132") (unit 1)
-        )
-      )
-    )
-  )
   (symbol (lib_id "Device:L_Small") (at 307.975 33.655 90) (unit 1)
     (in_bom yes) (on_board yes) (dnp no) (fields_autoplaced)
@@
     )
   )
-  (symbol (lib_id "Power_Protection:USBLC6-2SC6") (at 118.745 71.755 0) (unit 1)
-    (in_bom yes) (on_board yes) (dnp no)
-    (property "Reference" "U6" (at 123.825 62.865 0)
-      (effects (font (size 1.27 1.27)) (justify left))
-    )
-    (property "Value" "USBLC6-2SC6" (at 120.015 81.28 0)
-      (effects (font (size 1.27 1.27)) (justify left))
-    )
-    (property "Footprint" "Package_TO_SOT_SMD:SOT-23-6" (at 118.745 84.455 0)
-      (effects (font (size 1.27 1.27)) hide)
-    )
-    (property "Datasheet" "https://www.st.com/resource/en/datasheet/usblc6-2.pdf" (at 123.825 62.865 0)
-      (effects (font (size 1.27 1.27)) hide)
-    )
-    (pin "1")
-    (pin "2")
-    (pin "3")
-    (pin "4")
-    (pin "5")
-    (pin "6")
-    (instances
-      (project "wordclock-proto-r1"
-        (path "/4f94f353-fcb1-446a-8ea4-44fbed72b7d1"
-          (reference "U6") (unit 1)
-        )
-      )
-    )
-  )
   (symbol (lib_id "power:GND") (at 184.785 35.56 0) (unit 1)
     (in_bom yes) (on_board yes) (dnp no)
@@
         )
       )
-    )
-  )
-  (symbol (lib_id "power:+5V") (at 118.745 59.69 0) (unit 1)
-    (in_bom yes) (on_board yes) (dnp no) (fields_autoplaced)
-    (property "Reference" "#PWR0139" (at 118.745 63.5 0)
-      (effects (font (size 1.27 1.27)) hide)
-    )
-    (property "Value" "+5V" (at 118.745 55.88 0)
-      (effects (font (size 1.27 1.27)))
-    )
-    (property "Footprint" "" (at 118.745 59.69 0)
-      (effects (font (size 1.27 1.27)) hide)
-    )
-    (property "Datasheet" "" (at 118.745 59.69 0)
-      (effects (font (size 1.27 1.27)) hide)
-    )
-    (pin "1")
-    (instances
-      (project "wordclock-proto-r1"
-        (path "/4f94f353-fcb1-446a-8ea4-44fbed72b7d1"
-          (reference "#PWR0139") (unit 1)
-        )
-      )
