File: schematics/circuit/wordclock-r1/led_array.kicad_sch (KiCad schematic)
At the start: 67 parts, among them U2 MAX7219

Commit message: PCB 0.1 Changes (#4)
* Initial 16x16 wordclock layout

* Change tracked files

* Initial pcb layout

* Add prototype board project

* more pcb changes
Parts:
- renumbered C11 to C19, R2 to R13, U2 to U1
Connections:
- net VDD renamed +3.3V
